File: PCB/FCU_Power.kicad_sch (KiCad schematic)
At the start: 12 parts, among them U2 AP62300WU, U3 AP2112K-3.3

Commit message: Added MCU interfaces and started sensor design
Parts:
- R5: renamed from R1; value 52.3k -> 52k3
- renumbered C6 to C10, C7 to C11, C8 to C12, C11 to C13, C10 to C14, C9 to C8, C5 to C9, R2 to R6
Changed lines of the file:
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@@
 		(dnp no)
 		(fields_autoplaced yes)
-		(property "Reference" "C8"
+		(property "Reference" "C12"
 			(at 148.59 73.6599 0)
 			(show_name no)
@@
 			(project "STM32_FCU"
 				(path "/9fd53907-6a99-448d-8671-d17de9d6fa45/7272a036-0cd8-4a4f-a895-6bfae3d56c11"
-					(reference "C8")
+					(reference "C12")
 					(unit 1)
 				)
@@
 		(dnp no)
 		(fields_autoplaced yes)
-		(property "Reference" "#PWR09"
+		(property "Reference" "#PWR012"
 			(at 161.29 54.61 0)
 			(hide yes)
@@
 			(project "STM32_FCU"
 				(path "/9fd53907-6a99-448d-8671-d17de9d6fa45/7272a036-0cd8-4a4f-a895-6bfae3d56c11"
-					(reference "#PWR09")
+					(reference "#PWR012")
 					(unit 1)
 				)
@@
 		(dnp no)
 		(fields_autoplaced yes)
-		(property "Reference" "C6"
+		(property "Reference" "C10"
 			(at 110.49 72.3899 0)
 			(show_name no)
@@
 			(project "STM32_FCU"
 				(path "/9fd53907-6a99-448d-8671-d17de9d6fa45/7272a036-0cd8-4a4f-a895-6bfae3d56c11"
-					(reference "C6")
+					(reference "C10")
 					(unit 1)
 				)
@@
 		(dnp no)
 		(fields_autoplaced yes)
-		(property "Reference" "#PWR06"
+		(property "Reference" "#PWR010"
 			(at 116.84 99.06 0)
 			(hide yes)
@@
 			(project "STM32_FCU"
 				(path "/9fd53907-6a99-448d-8671-d17de9d6fa45/7272a036-0cd8-4a4f-a895-6bfae3d56c11"
-					(reference "#PWR06")
+					(reference "#PWR010")
 					(unit 1)
 				)
@@
 		(dnp no)
 		(fields_autoplaced yes)
-		(property "Reference" "R1"
+		(property "Reference" "R5"
 			(at 119.38 72.3899 0)
 			(show_name no)
@@
 			)
 		)
-		(property "Value" "52.3k"
+		(property "Value" "52k3"
 			(at 119.38 74.9299 0)
 			(show_name no)
@@
 			(project "STM32_FCU"
 				(path "/9fd53907-6a99-448d-8671-d17de9d6fa45/7272a036-0cd8-4a4f-a895-6bfae3d56c11"
-					(reference "R1")
+					(reference "R5")
 					(unit 1)
 				)
@@
 		(dnp no)
 		(fields_autoplaced yes)
-		(property "Reference" "#PWR07"
+		(property "Reference" "#PWR011"
 			(at 138.43 92.71 0)
 			(hide yes)
@@
 			(project "STM32_FCU"
 				(path "/9fd53907-6a99-448d-8671-d17de9d6fa45/7272a036-0cd8-4a4f-a895-6bfae3d56c11"
-					(reference "#PWR07")
+					(reference "#PWR011")
 					(unit 1)
 				)
@@
 		(dnp no)
 		(fields_autoplaced yes)
-		(property "Reference" "#PWR011"
+		(property "Reference" "#PWR013"
 			(at 215.9 91.44 0)
 			(hide yes)
@@
 			(project "STM32_FCU"
 				(path "/9fd53907-6a99-448d-8671-d17de9d6fa45/7272a036-0cd8-4a4f-a895-6bfae3d56c11"
-					(reference "#PWR011")
+					(reference "#PWR013")
 					(unit 1)
 				)
@@
 		(dnp no)
 		(fields_autoplaced yes)
-		(property "Reference" "C10"
+		(property "Reference" "C14"
 			(at 238.76 72.3899 0)
 			(show_name no)
@@
 			(project "STM32_FCU"
 				(path "/9fd53907-6a99-448d-8671-d17de9d6fa45/7272a036-0cd8-4a4f-a895-6bfae3d56c11"
-					(reference "C10")
+					(reference "C14")
 					(unit 1)
 				)
@@
 		(dnp no)
 		(fields_autoplaced yes)
-		(property "Reference" "C9"
+		(property "Reference" "C8"
 			(at 41.91 62.2299 0)
 			(show_name no)
@@
 			(project "STM32_FCU"
 				(path "/9fd53907-6a99-448d-8671-d17de9d6fa45/7272a036-0cd8-4a4f-a895-6bfae3d56c11"
-					(reference "C9")
+					(reference "C8")
 					(unit 1)
 				)
@@
 		(dnp no)
 		(fields_autoplaced yes)
-		(property "Reference" "#PWR05"
+		(property "Reference" "#PWR09"
 			(at 72.39 96.52 0)
 			(hide yes)
@@
 			(project "STM32_FCU"
 				(path "/9fd53907-6a99-448d-8671-d17de9d6fa45/7272a036-0cd8-4a4f-a895-6bfae3d56c11"
-					(reference "#PWR05")
+					(reference "#PWR09")
 					(unit 1)
 				)
@@
 		(dnp no)
 		(fields_autoplaced yes)
-		(property "Reference" "R2"
+		(property "Reference" "R6"
 			(at 119.38 85.0899 0)
 			(show_name no)
@@
 			(project "STM32_FCU"
 				(path "/9fd53907-6a99-448d-8671-d17de9d6fa45/7272a036-0cd8-4a4f-a895-6bfae3d56c11"
-					(reference "R2")
+					(reference "R6")
 					(unit 1)
 				)
@@
 		(dnp no)
 		(fields_autoplaced yes)
-		(property "Reference" "C11"
+		(property "Reference" "C13"
 			(at 200.66 72.3899 0)
 			(show_name no)
@@
 			(project "STM32_FCU"
 				(path "/9fd53907-6a99-448d-8671-d17de9d6fa45/7272a036-0cd8-4a4f-a895-6bfae3d56c11"
-					(reference "C11")
+					(reference "C13")
 					(unit 1)
 				)
@@
 		(dnp no)
 		(fields_autoplaced yes)
-		(property "Reference" "C5"
+		(property "Reference" "C9"
 			(at 90.17 62.2299 0)
 			(show_name no)
@@
 			(project "STM32_FCU"
 				(path "/9fd53907-6a99-448d-8671-d17de9d6fa45/7272a036-0cd8-4a4f-a895-6bfae3d56c11"
-					(reference "C5")
+					(reference "C9")
 					(unit 1)
 				)
@@
 		(dnp no)
 		(fields_autoplaced yes)
-		(property "Reference" "C7"
+		(property "Reference" "C11"
 			(at 135.89 73.6599 0)
 			(show_name no)
@@
 			(project "STM32_FCU"
 				(path "/9fd53907-6a99-448d-8671-d17de9d6fa45/7272a036-0cd8-4a4f-a895-6bfae3d56c11"
-					(reference "C7")
+					(reference "C11")
 					(unit 1)
 				)
@@
 		(dnp no)
 		(fields_autoplaced yes)
-		(property "Reference" "#PWR04"
+		(property "Reference" "#PWR07"
 			(at 33.02 54.61 0)
 			(hide yes)
@@
 			(project "STM32_FCU"
 				(path "/9fd53907-6a99-448d-8671-d17de9d6fa45/7272a036-0cd8-4a4f-a895-6bfae3d56c11"
-					(reference "#PWR04")
+					(reference "#PWR07")
 					(unit 1)
 				)
@@
 		(dnp no)
 		(fields_autoplaced yes)
-		(property "Reference" "#PWR012"
+		(property "Reference" "#PWR014"
 			(at 241.3 69.85 0)
 			(hide yes)
@@
 			(project "STM32_FCU"
 				(path "/9fd53907-6a99-448d-8671-d17de9d6fa45/7272a036-0cd8-4a4f-a895-6bfae3d56c11"
-					(reference "#PWR012")
-					(unit 1)
-				)
+					(reference "#PWR014")
+					(unit 1)
+				)
